File: OpenLTTO Barrel Module.kicad_sch (KiCad schematic)
At the start: 16 parts, among them Q1 IRLML6244, U1 TSOP4138

Commit message: Updated schematic metadata, added schematic PDF and renders of PCB
Other:
- company: (none) -> Paul Mumby
- title: (none) -> OpenLTTO Barrel Module
Changed lines of the file:
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@@
 (kicad_sch (version 20230121) (generator eeschema)
   (paper "A4")
+  (title_block
+    (title "OpenLTTO Barrel Module")
+    (rev "1.0")
+    (company "Paul Mumby")
+  )
   (junction (at 107.95 134.62) (diameter 0) (color 0 0 0 0)
   )
